Commit message: Adding Assignment-2

File: src/diff_drive_description/urdf/diff_drive.urdf (robot description, URDF)
Before this commit: robot RoboBot, 3 links, 2 joints
Links:
- added link camera1, mass 1e-5; collision box size=0.025 0.025 0.025; visual box size=0.025 0.025 0.025
- added link camera2, mass 1e-5; collision box size=0.025 0.025 0.025; visual box size=0.025 0.025 0.025
- added link hokuyo_link, mass 1e-5; collision box size=0.03 0.03 0.03; visual box size=0.03 0.03 0.03
Joints:
- added joint camera1_joint: type fixed, parent chassis, child camera1, origin xyz=0.25 0.1 0 rpy=0 0 0, axis 0 1 0
- added joint camera2_joint: type fixed, parent chassis, child camera2, origin xyz=0.25 -0.1 0 rpy=0 0 0, axis 0 1 0
- added joint hokuyo_joint: type fixed, parent chassis, child hokuyo_link, origin xyz=0 0 0.125 rpy=0 0 0, axis 0 1 0
